Commit message: added ft sensor in urdf

File: fh_desc/model.urdf (robot description, URDF)
Before this commit: robot smart_grasping_sandbox, 35 links, 34 joints
Joints:
- joint H1_F1_tip: limit (none) -> lower=0 upper=0 effort=10 velocity=1; type fixed -> revolute
- joint H1_F1_tip_to_optoforce: axis (none) -> 1 0 0; limit (none) -> lower=0 upper=0 effort=10 velocity=1; type fixed -> revolute

Commit message: added force/torque on H1J3 joint

File: fh_desc/model.urdf (robot description, URDF)
Before this commit: robot smart_grasping_sandbox, 35 links, 34 joints
Joints:
- joint H1_F1_tip: limit lower=0 upper=0 effort=10 velocity=1 -> (none); origin (none) -> xyz=0 0 0 rpy=0 0 0; type revolute -> fixed
- joint H1_F1_tip_to_optoforce: axis 1 0 0 -> (none); limit lower=0 upper=0 effort=10 velocity=1 -> (none); type revolute -> fixed
